Commit message: Gezebo

File: ros_parol/src/parol6/urdf/parol6.urdf (robot description, URDF)
Before this commit: robot parol6, 8 links, 7 joints
Links:
- link L6: mass 0.0703261410665101 -> 0.4156; geometry collision mesh filename=package://parol6/meshes/L6.STL scale=0.001 0.001 0.001; visual mesh filename=package://parol6/meshes/L6.STL scale=0.001 0.001 0.001
Joints:
- removed joint L1
- removed joint L2
- removed joint L3
- removed joint L4
- removed joint L5
- removed joint L6
- added joint joint_1: type revolute, parent base_link, child L1, origin xyz=0 0 0 rpy=0 0 0, axis 0 0 1, limit lower=-1.7 upper=1.7 effort=300 velocity=3
- added joint joint_2: type revolute, parent L1, child L2, origin xyz=0.0234207210610375 0 0.1105 rpy=-1.5707963267949 0 0, axis 0 0 1, limit lower=-0.98 upper=1 effort=300 velocity=3
- added joint joint_3: type revolute, parent L2, child L3, origin xyz=0 -0.18 0 rpy=3.1416 0 -1.5708, axis 0 0 -1, limit lower=-2 upper=1.3 effort=300 velocity=3
- added joint joint_4: type revolute, parent L3, child L4, origin xyz=0.0435 0 0 rpy=1.5707963267949 0 3.14159265358979, axis 0 0 -1, limit lower=-2 upper=2 effort=300 velocity=3
- added joint joint_5: type revolute, parent L4, child L5, origin xyz=0 0 -0.17635 rpy=-1.5708 0 0, axis 0 0 -1, limit lower=-2.1 upper=2.1 effort=300 velocity=3
- added joint joint_6: type continuous, parent L5, child L6, origin xyz=0 0.077 0 rpy=1.5708 0 0, axis 0 0 -1, limit lower=-3.1 upper=3.1 effort=300 velocity=3

File: ros_parol/src/parol6_moveit/config/parol6.ros2_control.xacro (robot description, xacro)
@@ -6,7 +6,7 @@
             <hardware>
                 <!-- By default, set up controllers for simulation. This won't work on real hardware -->
-                <plugin>mock_components/GenericSystem</plugin>
+                <plugin>gazebo_ros2_control/GazeboSystem</plugin>
             </hardware>
-            <joint name="L1">
+            <joint name="joint_1">
                 <command_interface name="position"/>
                 <state_interface name="position">
@@ -15,5 +15,5 @@
                 <state_interface name="velocity"/>
             </joint>
-            <joint name="L2">
+            <joint name="joint_2">
                 <command_interface name="position"/>
                 <state_interface name="position">
@@ -22,5 +22,5 @@
                 <state_interface name="velocity"/>
             </joint>
-            <joint name="L3">
+            <joint name="joint_3">
                 <command_interface name="position"/>
                 <state_interface name="position">
@@ -29,5 +29,5 @@
                 <state_interface name="velocity"/>
             </joint>
-            <joint name="L4">
+            <joint name="joint_4">
                 <command_interface name="position"/>
                 <state_interface name="position">
@@ -36,5 +36,5 @@
                 <state_interface name="velocity"/>
             </joint>
-            <joint name="L5">
+            <joint name="joint_5">
                 <command_interface name="position"/>
                 <state_interface name="position">
@@ -43,5 +43,5 @@
                 <state_interface name="velocity"/>
             </joint>
-            <joint name="L6">
+            <joint name="joint_6">
                 <command_interface name="position"/>
                 <state_interface name="position">

Commit message: Gazebo + MoveIt2 setting

File: ros_parol/src/parol6/urdf/parol6.urdf (robot description, URDF)
Before this commit: robot parol6, 8 links, 7 joints
Links:
- link L6: geometry collision mesh filename=package://parol6/meshes/L6.STL; visual mesh filename=package://parol6/meshes/L6.STL

File: ros_parol/src/parol6_moveit/config/parol6.ros2_control.xacro (robot description, xacro)
@@ -1,10 +1,14 @@
 <?xml version="1.0"?>
 <robot xmlns:xacro="http://www.ros.org/wiki/xacro">
-    <xacro:macro name="parol6_ros2_control" params="name initial_positions_file">
-        <xacro:property name="initial_positions" value="${load_yaml(initial_positions_file)['initial_positions']}"/>
+    <xacro:macro name="parol6_ros2_control" params="name initial_positions_file sim_mode">
+        <xacro:property name="initial_positions" value="${xacro.load_yaml(initial_positions_file)['initial_positions']}"/>
         <ros2_control name="${name}" type="system">
             <hardware>
-                <!-- By default, set up controllers for simulation. This won't work on real hardware -->
-                <plugin>gazebo_ros2_control/GazeboSystem</plugin>
+                <xacro:if value="${sim_mode == 'gz'}">
+                    <plugin>gz_ros2_control/GazeboSimSystem</plugin>
+                </xacro:if>
+                <xacro:if value="${sim_mode == 'mock'}">
+                    <plugin>mock_components/GenericSystem</plugin>
+                </xacro:if>
             </hardware>
             <joint name="joint_1">
@@ -51,4 +55,11 @@
             </joint>
         </ros2_control>
+        <xacro:if value="${sim_mode == 'gz'}">
+            <gazebo>
+                <plugin filename="gz_ros2_control-system" name="gz_ros2_control::GazeboSimROS2ControlPlugin">
+                    <parameters>$(find parol6_moveit)/config/ros2_controllers.yaml</parameters>
+                </plugin>
+            </gazebo>
+        </xacro:if>
     </xacro:macro>
 </robot>

File: ros_parol/src/parol6_moveit/config/parol6.urdf.xacro (robot description, xacro)
@@ -2,8 +2,23 @@
 <robot xmlns:xacro="http://www.ros.org/wiki/xacro" name="parol6">
     <xacro:arg name="initial_positions_file" default="initial_positions.yaml" />
+    <!--
+        sim_mode controls which ros2_control hardware plugin gets injected by
+        parol6.ros2_control.xacro:
+            mock  -> mock_components/GenericSystem (used by demo.launch.py via
+                     the MoveIt-Setup-Assistant-generated rsp/move_group/etc.
+                     sub-launches, which all read this default)
+            gz    -> gz_ros2_control/GazeboSimSystem + the gz_ros2_control-system
+                     plugin tag (set explicitly by gazebo.launch.py)
+        Default is mock because the sub-launches in generate_demo_launch each
+        rebuild MoveItConfigsBuilder from scratch and only see the default.
+    -->
+    <xacro:arg name="sim_mode" default="mock" />
     <!-- Import parol6 urdf file -->
     <xacro:include filename="$(find parol6)/urdf/parol6.urdf" />
     <!-- Import control_xacro -->
     <xacro:include filename="parol6.ros2_control.xacro" />
-    <xacro:parol6_ros2_control name="FakeSystem" initial_positions_file="$(arg initial_positions_file)"/>
+    <xacro:parol6_ros2_control
+        name="GazeboSystem"
+        initial_positions_file="$(arg initial_positions_file)"
+        sim_mode="$(arg sim_mode)"/>
 </robot>
